Commit message: Update

File: description/robot_core.xacro (robot description, xacro)
@@ -1,3 +1,7 @@
 <?xml version="1.0"?>
 <robot xmlns:xacro="http://www.ros.org/wiki/xacro">
+    <xacro:include filename="color.xacro" />
+    <!-- Base Link -->
+    <link name="base_link">
+    </link>
 </robot>

Commit message: update

File: description/robot_core.xacro (robot description, xacro)
@@ -5,3 +5,18 @@
     <link name="base_link">
     </link>
+    <!-- Chassis Joint -->
+    <joint name="chassis_joint" type="fixed">
+        <parent link="base_link" />
+        <child link="chassis" />
+        <origin xyz="0 0 0" />
+    </joint>
+    <!-- Chassis Link -->
+    <link name="chassis">
+        <visual>
+            <origin xyz="0 0 0.05" rpy="0 0 0"/>
+            <geometry>
+                <box size="0.15 0.15 0.15"/>
+            </geometry>
+            <material name="white" />
+        </visual>
 </robot>
